File: test/pcbs/mock_footprints___pcbs_main.kicad_pcb (KiCad board)
At the start: 2 copper layers, 39 x 19 mm, 8 parts

Commit message: New Kicad format plus tests
Parts:
- removed the ? at (0.00, 0.00) (x4)
- added ?: , anchor_test, F.Cu at (0.00, 0.00)
Changed lines of the file:
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@@
-(kicad_pcb (version 20171130) (host pcbnew 5.1.6)
-  (page A3)
+(kicad_pcb (version 20211014) (generator pcbnew)
+  (general
+    (thickness 1.6)
+  )
+  (paper "A3")
   (title_block
     (title main)
@@
     (company Unknown)
   )
-  (general
-    (thickness 1.6)
-  )
   (layers
-    (0 F.Cu signal)
-    (31 B.Cu signal)
-    (32 B.Adhes user)
-    (33 F.Adhes user)
-    (34 B.Paste user)
-    (35 F.Paste user)
-    (36 B.SilkS user)
-    (37 F.SilkS user)
-    (38 B.Mask user)
-    (39 F.Mask user)
-    (40 Dwgs.User user)
-    (41 Cmts.User user)
-    (42 Eco1.User user)
-    (43 Eco2.User user)
-    (44 Edge.Cuts user)
-    (45 Margin user)
-    (46 B.CrtYd user)
-    (47 F.CrtYd user)
-    (48 B.Fab user)
-    (49 F.Fab user)
+    (0 "F.Cu" signal)
+    (31 "B.Cu" signal)
+    (32 "B.Adhes" user "B.Adhesive")
+    (33 "F.Adhes" user "F.Adhesive")
+    (34 "B.Paste" user)
+    (35 "F.Paste" user)
+    (36 "B.SilkS" user "B.Silkscreen")
+    (37 "F.SilkS" user "F.Silkscreen")
+    (38 "B.Mask" user)
+    (39 "F.Mask" user)
+    (40 "Dwgs.User" user "User.Drawings")
+    (41 "Cmts.User" user "User.Comments")
+    (42 "Eco1.User" user "User.Eco1")
+    (43 "Eco2.User" user "User.Eco2")
+    (44 "Edge.Cuts" user)
+    (45 "Margin" user)
+    (46 "B.CrtYd" user "B.Courtyard")
+    (47 "F.CrtYd" user "F.Courtyard")
+    (48 "B.Fab" user)
+    (49 "F.Fab" user)
   )
   (setup
@@
     (visible_elements FFFFFF7F)
     (pcbplotparams
-      (layerselection 0x010fc_ffffffff)
+      (layerselection 0x00010fc_ffffffff)
+      (disableapertmacros false)
       (usegerberextensions false)
       (usegerberattributes true)
       (usegerberadvancedattributes true)
       (creategerberjobfile true)
+      (svguseinch false)
+      (svgprecision 6)
       (excludeedgelayer true)
-      (linewidth 0.100000)
       (plotframeref false)
       (viasonmask false)
@@
       (hpglpenspeed 20)
       (hpglpendiameter 15.000000)
+      (dxfpolygonmode true)
+      (dxfimperialunits true)
+      (dxfusepcbnewfont true)
       (psnegative false)
       (psa4output false)
@@
       (plotvalue true)
       (plotinvisibletext false)
-      (padsonsilk false)
+      (sketchpadsonfab false)
       (subtractmaskfromsilk false)
       (outputformat 1)
@@
       (drillshape 1)
       (scaleselection 1)
-      (outputdirectory ""))
+      (outputdirectory "")
+    )
   )
             (net 0 "")
@@
                     (fp_line (start 0 0) (end 10 -10) (layer Dwgs.User) (width 0.05))
                 )
-                (module anchor_test (layer F.Cu)
-                    (at 0 0 0)
-                    (fp_line (start 0 0) (end 0 0) (layer Dwgs.User) (width 0.05))
-                )
-                (module arrobj_test (layer F.Cu)
-                    (at 0 0 0)
-                    (fp_line (start 5 5) (end 6 6) (layer Dwgs.User) (width 0.05))
-(fp_line (start 5 5) (end 7 7) (layer Dwgs.User) (width 0.05))
-                )
-                (module arrobj_test (layer F.Cu)
-                    (at 0 0 0)
-                    (fp_line (start 5 5) (end 6 6) (layer Dwgs.User) (width 0.05))
-(fp_line (start 5 5) (end 7 5) (layer Dwgs.User) (width 0.05))
-                )
-            (gr_line (start -9.5 9.5) (end 9.5 9.5) (angle 90) (layer Edge.Cuts) (width 0.15))
-(gr_line (start 9.5 9.5) (end 9.5 -9.5) (angle 90) (layer Edge.Cuts) (width 0.15))
-(gr_line (start 9.5 -9.5) (end -9.5 -9.5) (angle 90) (layer Edge.Cuts) (width 0.15))
-(gr_line (start -9.5 -9.5) (end -9.5 9.5) (angle 90) (layer Edge.Cuts) (width 0.15))
-(gr_line (start 10.5 9.5) (end 29.5 9.5) (angle 90) (layer Edge.Cuts) (width 0.15))
-(gr_line (start 29.5 9.5) (end 29.5 -9.5) (angle 90) (layer Edge.Cuts) (width 0.15))
-(gr_line (start 29.5 -9.5) (end 10.5 -9.5) (angle 90) (layer Edge.Cuts) (width 0.15))
-(gr_line (start 10.5 -9.5) (end 10.5 9.5) (angle 90) (layer Edge.Cuts) (width 0.15))
+            (gr_line (start -9.5 9.5) (end 9.5 9.5) (layer "Edge.Cuts") (width 0.15))
+(gr_line (start 9.5 9.5) (end 9.5 -9.5) (layer "Edge.Cuts") (width 0.15))
+(gr_line (start 9.5 -9.5) (end -9.5 -9.5) (layer "Edge.Cuts") (width 0.15))
+(gr_line (start -9.5 -9.5) (end -9.5 9.5) (layer "Edge.Cuts") (width 0.15))
+(gr_line (start 10.5 9.5) (end 29.5 9.5) (layer "Edge.Cuts") (width 0.15))
+(gr_line (start 29.5 9.5) (end 29.5 -9.5) (layer "Edge.Cuts") (width 0.15))
+(gr_line (start 29.5 -9.5) (end 10.5 -9.5) (layer "Edge.Cuts") (width 0.15))
+(gr_line (start 10.5 -9.5) (end 10.5 9.5) (layer "Edge.Cuts") (width 0.15))
 )
